File: receiver/receiver.kicad_sch (KiCad schematic)
At the start: 72 parts, among them J1 USB_B_Mini, J2 Conn_01x04_Pin, J3 Conn_01x04_Pin, SW1 SW_Push, SW2 SW_SPDT, U1 AMS1117-3.3, U2 STM32F303K8Tx, U3 MAX2622, U4 HMC356, U5 LT5517, U6 MABAES0054, U7 FT232RL, Y1 16MHz

Commit message: Final version
Parts:
- removed C17: 2.2u, Capacitor_SMD:C_0603_1608Metric_Pad1.08x0.95mm_HandSolder, symbol Device:C
- C11: value C -> 1n
- C2: value C -> 2p
- C4, C8: value C -> 10p
- C7: value C -> 0.1p
- J2: value Conn_01x04_Pin -> UART
- J3: value Conn_01x04_Pin -> SWD
- L1, L2: value L -> 8.2n
- R13, R14: value 1k -> 10k
- R3: value 1k5 -> 10k
Connections:
- net ADC2_IN1: now reaches U2.10 (PA4)
- net ADC2_IN2: now reaches U2.11 (PA5)
- no-connect marks 37 -> 35
Other:
- note added: "https://www.mouser.pl/ProductDetail/MACOM/MABA-010268-CT4160?qs=doiCPypUmgEbCViX1mrIng%3D%3D"
- note added: "max 2.37 V min 0 V"
- note removed: "Filtr kwadratowy o połowe którszy np. Czebyszew. jakimś kalkulatorem, zrobić większy bandwidth. 1M 10 razy większy niż ten w transiverze."
- note removed: "https://www.digikey.in/en/products/detail/531BC866M000DG/16345803"
- moved on the sheet: C1, C4, C5, L1, Y1
