File: transmiter/transmiter.kicad_pcb (KiCad board)
At the start: 2 copper layers, 55 x 57 mm, 73 parts, among them J1 USB_B_Mini, J2 Conn_01x04_Pin, J3 Conn_01x04_Pin, SW1 SW_Push, SW2 SW_SPDT, U1 ADL5370, U2 MAX2608, U3 AMS1117-3.3, U4 ADL5531, U6 FIN1001M5X, U7 FIN1001M5X, U8 STM32F303K8Tx, U9 FT232RL, Y1 16MHz

Commit message: Final version
Parts:
- C1, C3: value 20p -> 10p
- C12: value 22u -> 10u
- C2: value 0.1u -> 100n
- C27, C32: value C -> 220p
- C9: value 22u -> 100n
- J2: value Conn_01x04_Pin -> UART
- J3: value Conn_01x04_Pin -> SWD
- L1, L2, L3, L4: value 80u -> 100u
- R10, R4: value 1k5 -> 1k
- R11: value 1.5k -> 1k
- moved C7 15.4 mm to (98.3, 64.4)
- moved C5 15.4 mm to (109.4, 75.1)
Connections:
- C15 pad 1: Net-(U1-LOIP) -> LO_P
- C15 pad 2: LO_P -> Net-(U1-LOIP)
- C16 pad 1: Net-(U1-LOIN) -> LO_N
- C16 pad 2: LO_N -> Net-(U1-LOIN)
