File: transmiter/transmiter.kicad_sch (KiCad schematic)
At the start: 73 parts, among them J1 USB_B_Mini, J2 Conn_01x04_Pin, J3 Conn_01x04_Pin, SW1 SW_Push, SW2 SW_SPDT, U1 ADL5370, U2 MAX2608, U3 AMS1117-3.3, U4 ADL5531, U6 FIN1001M5X, U7 FIN1001M5X, U8 STM32F303K8Tx, U9 FT232RL, Y1 16MHz

Commit message: Final version
Parts:
- J2: value Conn_01x04_Pin -> UART
- J3: value Conn_01x04_Pin -> SWD
- L5: value 470n -> 390n
Other:
- note added: "https://www.digikey.pl/en/products/MAX2608"
- note removed: "https://www.digikey.pl/en/products/MAX2608EUT-T"
- moved on the sheet: C32
Changed lines of the file:
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@@
 	(wire
 		(pts
+			(xy 172.72 148.59) (xy 172.72 146.05)
+		)
+		(stroke
+			(width 0)
+			(type default)
+		)
+	)
+	(wire
+		(pts
 			(xy 31.75 148.59) (xy 41.91 148.59)
 		)
@@
 	(wire
 		(pts
-			(xy 172.72 135.89) (xy 172.72 137.16)
+			(xy 172.72 135.89) (xy 172.72 138.43)
 		)
 		(stroke
@@
 		)
 	)
-	(text "https://www.digikey.pl/en/products/MAX2608EUT-T"
+	(text "https://www.digikey.pl/en/products/MAX2608\n"
 		(exclude_from_sim no)
-		(at 183.896 156.21 0)
+		(at 181.61 157.226 0)
 		(effects
 			(font
@@
 	(text "https://www.tme.eu/pl/ft232rl-reel/"
 		(exclude_from_sim no)
-		(at 120.142 70.866 0)
+		(at 120.396 70.358 0)
 		(effects
 			(font
@@
 	(text "https://botland.com.pl/usb-uart.html"
 		(exclude_from_sim no)
-		(at 120.65 73.66 0)
+		(at 120.904 73.152 0)
 		(effects
 			(font
@@
 	(symbol
 		(lib_id "Device:C")
-		(at 172.72 140.97 180)
+		(at 172.72 142.24 180)
 		(unit 1)
 		(exclude_from_sim no)
@@
 		(dnp no)
 		(property "Reference" "C32"
-			(at 165.608 139.954 0)
+			(at 165.608 141.224 0)
 			(effects
 				(font
@@
 		)
 		(property "Value" "220p"
-			(at 165.608 142.494 0)
+			(at 165.608 143.764 0)
 			(effects
 				(font
@@
 		)
 		(property "Footprint" "Capacitor_SMD:C_0603_1608Metric_Pad1.08x0.95mm_HandSolder"
-			(at 171.7548 137.16 0)
+			(at 171.7548 138.43 0)
 			(effects
 				(font
@@
 		)
 		(property "Datasheet" "~"
-			(at 172.72 140.97 0)
+			(at 172.72 142.24 0)
 			(effects
 				(font
@@
 		)
 		(property "Description" "Unpolarized capacitor"
-			(at 172.72 140.97 0)
+			(at 172.72 142.24 0)
 			(effects
 				(font
@@
 			)
 		)
-		(property "Value" "470n"
+		(property "Value" "390n"
 			(at 247.65 38.0999 0)
 			(effects
@@
 			)
 		)
-		(property "Value" "Conn_01x04_Pin"
+		(property "Value" "UART"
 			(at 133.985 143.51 0)
 			(effects
@@
 			)
 		)
-		(property "Value" "Conn_01x04_Pin"
+		(property "Value" "SWD"
 			(at 111.125 143.51 0)
 			(effects
@@
 	(symbol
 		(lib_id "power:GND")
-		(at 172.72 144.78 0)
+		(at 172.72 148.59 0)
 		(unit 1)
 		(exclude_from_sim no)
@@
 		(fields_autoplaced yes)
 		(property "Reference" "#PWR053"
-			(at 172.72 151.13 0)
+			(at 172.72 154.94 0)
 			(effects
 				(font
@@
 		)
 		(property "Value" "GND"
-			(at 172.72 149.86 0)
+			(at 172.72 153.67 0)
 			(effects
 				(font
@@
 		)
 		(property "Footprint" ""
-			(at 172.72 144.78 0)
+			(at 172.72 148.59 0)
 			(effects
 				(font
@@
 		)
 		(property "Datasheet" ""
-			(at 172.72 144.78 0)
+			(at 172.72 148.59 0)
 			(effects
 				(font
@@
 		)
 		(property "Description" "Power symbol creates a global label with name \"GND\" , ground"
-			(at 172.72 144.78 0)
+			(at 172.72 148.59 0)
 			(effects
 				(font
